File: rack/thatmicpre_v2.kicad_sch (KiCad schematic)
At the start: 89 parts, among them J1 CON-SOCJ-2155, J10 Conn_01x03_Female, J2 NC3FBH1, J3 NC3MBH1, J4 Conn_01x03_Female, J5 Conn_01x03_Male, J6 Conn_01x04_Female, J7 Conn_01x04_Male, J8 Conn_01x04_Female, J9 NMJ6HFD2, Q1 BC546CTA, Q2 BC546CTA, SW1 PBH2UEESNPNAGX, SW2 PBH2UEESNPNAGX, SW3 SR2612F-0112-38F5B-D8-S, U1 THAT1510P08-U

Commit message: Production version of v2.0 (rack version) with panels
Parts:
- removed J10: Conn_01x03_Female, Connector_PinHeader_2.54mm:PinHeader_1x03_P2.54mm_Vertical, symbol Connector:Conn_01x03_Female
- removed J2: NC3FBH1, Connector_Audio:Jack_XLR_Neutrik_NC3FBH1_Horizontal, symbol Connector:XLR3
- removed J3: NC3MBH1, Connector_Audio:Jack_XLR_Neutrik_NC3MBH_Horizontal, symbol Connector:XLR3
- removed J4: Conn_01x03_Female, Connector_PinSocket_2.54mm:PinSocket_1x03_P2.54mm_Horizontal, symbol Connector:Conn_01x03_Female
- removed J5: Conn_01x03_Male, Connector_PinHeader_2.54mm:PinHeader_1x03_P2.54mm_Vertical, symbol Connector:Conn_01x03_Male
- removed J8: Conn_01x04_Female, Connector_PinHeader_2.54mm:PinHeader_1x04_P2.54mm_Vertical, symbol Connector:Conn_01x04_Female
- added D10, D11: LED, LED_THT:LED_D5.0mm, symbol Device:LED
- added J10, J8: Angled pinheader, Connector_PinHeader_2.54mm:PinHeader_1x04_P2.54mm_Vertical, symbol Connector:Conn_01x04_Male
- added J2: NC3FBH2, Connector_Audio:Jack_XLR_Neutrik_NC3FBH2_Horizontal, symbol Connector:XLR3_Ground
- added J3: NC3MBH1, Connector_Audio:Jack_XLR_Neutrik_NC3MBH_Horizontal, symbol Connector:XLR3_Ground
- added J4: Female header, Connector_PinSocket_2.54mm:PinSocket_1x04_P2.54mm_Horizontal, symbol Connector:Conn_01x04_Female
- added J5: Male pinheader, Connector_PinHeader_2.54mm:PinHeader_1x04_P2.54mm_Vertical, symbol Connector:Conn_01x04_Male
- J6: value Conn_01x04_Female -> Female header
- J7: value Conn_01x04_Male -> Male pinheader
- R27, R30: value 10k -> 47k; Vendor MBB02070C1002FCT00 -> MBB02070C4702FCT00
- SW1, SW2: value PBH2UEESNPNAGX -> DPDT; Vendor E-Switch -> PBH2UEEKZXNAG1RBLK
Connections:
- net GND: now also J10.2 (Pin_2), J10.3 (Pin_3), J2.1, J2.G, J3.1, J3.G, J4.2 (Pin_2), J4.3 (Pin_3)
- net at D6.2 (A), J6.3 (Pin_3), J6.4 (Pin_4)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: now also J8.3 (Pin_3), J8.4 (Pin_4)
- net at C2.1, C4.1, R6.2: now also J2.2
- net at C1.1, C5.1, R5.2: now also J2.3
- net at R10.2: now also J10.1 (Pin_1), J4.1 (Pin_1)
- net at C15.1, J9.T, R26.1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: now also J3.2
- net at C17.1, J9.R, R29.1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: now also J3.3
- net at C13.1, J6.1 (Pin_1), J6.2 (Pin_2): now also J8.1 (Pin_1), J8.2 (Pin_2)
- net at D9.3 (A2): now also D11.2 (A), J5.1 (Pin_1)
- net at D9.2 (K): now also D10.1 (K), D11.1 (K), J5.2 (Pin_2), J5.3 (Pin_3)
- net at D9.1 (A1): now also D10.2 (A), J5.4 (Pin_4)
- net at R11.2: now also J10.4 (Pin_4), J4.4 (Pin_4)
Other:
- note added: "L2,L3: Inductors, ferrites or 10R resistors"
- note added: "Mount either one dual-color LED, or two single LEDs."
- note added: "Mount either: 1. Angled female header on mainboard and straight male header on frontpanel. 2. Angled male pin header soldered to both mainboard and frontpanel."
- moved on the sheet: C5, D1, D15, D16, D18, D19, D2, D9, H1, H2, H3, H4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

Commit message: Modified rack version BOM to match assembled prototype
Parts:
- removed D10, D11: LED, LED_THT:LED_D5.0mm, symbol Device:LED
- C1, C2: Mfr Part Nr (none) -> FG28C0G2A471JNT0; Vendor RDE5C2A471J0M1H03A -> (none)
- C10, C11, C12, C7, C8: Mfr Part Nr (none) -> UPW1J221MPD; Vendor UPW1J221MPD -> (none)
- C13: Mfr Part Nr (none) -> UFW0J332MPD; Vendor UFW0J332MPD -> (none)
- C14, C16: value 22u-63V -> 22u-50V; Mfr Part Nr (none) -> UEP1V220MED
- C15, C17: Mfr Part Nr (none) -> PHE426DJ5100JR05; Vendor PHE426DJ5100JR05 -> (none)
- C18: value 1000u-25V -> 220u-63V; Mfr Part Nr (none) -> UPW1J221MPD; Vendor UVZ1E102MPD1CM -> (none)
- C3: Mfr Part Nr (none) -> FG28C0G2A470JNT0; Vendor RDE5C2A470J0M1H03A -> (none)
- C4, C5: Mfr Part Nr (none) -> UVP1J470MPD; Vendor UVP1J470MPD -> (none)
- C6: Mfr Part Nr (none) -> R82EC3100AA70J; Vendor R82EC3100AA70J -> (none)
- C9: Mfr Part Nr (none) -> R82EC3100AA70J; Vendor FG28X5R1E475KRT06 -> (none)
- D1, D2, D3, D4, D7: Mfr Part Nr (none) -> 1N4004GP; Vendor 1N4004GP-E3/54 -> (none)
- D13, D18, D19, D5, D6, D8: Mfr Part Nr (none) -> 1N4148; Vendor 1N4148 -> (none)
- D15, D16, D17: value 18V -> 16V; Mfr Part Nr (none) -> BZX55B16; Vendor BZX55B18-TAP -> (none)
- D9: Mfr Part Nr (none) -> WP59EGW
- F1: Mfr Part Nr (none) -> 0ZRC0015FF1E; Vendor Bel Fuse -> (none)
- J1: Mfr Part Nr (none) -> CON-SOCJ-2155
- J10, J8: Mfr Part Nr (none) -> TSW-104-08-F-S-RA
- J2: Mfr Part Nr (none) -> NC3FBH2
- J3: Mfr Part Nr (none) -> NC3MBH1
- J4, J6: Mfr Part Nr (none) -> SSQ-104-02-T-S-RA
- J5, J7: Mfr Part Nr (none) -> TSW-104-07-T-S
- J9: Mfr Part Nr (none) -> NMJ6HFD2
- L2, L3: value 4u7 -> 10u; Mfr Part Nr (none) -> 78F100J-TR-RC
- Q1: Cmp name BC546CTA -> (none); Mfr Part Nr (none) -> BC546CTA; Vendor BC546CTA -> (none)
- Q2: Mfr Part Nr (none) -> BC546CTA; Vendor BC546CTA -> (none)
- R1, R2: Mfr Part Nr (none) -> YR1B1K21CC; Vendor YR1B1K21CC -> (none)
- R10, R11, R7: Mfr Part Nr (none) -> MBB02070C2202FCT00; Vendor MBB02070C2202FCT00 -> (none)
- R13, R9: Mfr Part Nr (none) -> MBB02070C1002FCT00; Vendor MBB02070C1002FCT00 -> (none)
- R14: value 1M0 -> 8K06; Mfr Part Nr (none) -> MBB02070C1004FCT00; Vendor MBB02070C1004FCT00 -> (none)
- R15: value 2k7 -> 909R; Mfr Part Nr (none) -> MBB02070C2701FC100; Vendor MBB02070C2701FC100 -> (none)
- R16: value 1k0 -> 453R; Mfr Part Nr (none) -> MBB02070C1001FC100; Vendor MBB02070C1001FC100 -> (none)
- R17: value 560R -> 237R; Mfr Part Nr (none) -> MBB02070C5600FC100; Vendor MBB02070C5600FC100 -> (none)
- R18: value 270R -> 127R; Mfr Part Nr (none) -> MBB02070C2700FC100; Vendor MBB02070C2700FC100 -> (none)
- R19: value 150R -> 71R; Mfr Part Nr (none) -> MBB02070C1500FC100; Vendor MBB02070C1500FC100 -> (none)
- R20: value 82R -> 39R; Mfr Part Nr (none) -> MFR50SFTE52-82R; Vendor MFR50SFTE52-82R -> (none)
- R21: value 47R -> 22R; Mfr Part Nr (none) -> MFR50SFTE52-47R; Vendor MFR50SFTE52-47R -> (none)
- R22: value 27R -> 12R4; Mfr Part Nr (none) -> MFR50SFTE52-27R; Vendor MFR50SFTE52-27R -> (none)
- R23: value 15R -> 6R81; Mfr Part Nr (none) -> MFR50SFTE52-15R; Vendor MFR50SFTE52-15R -> (none)
- R24: value 8R2 -> 3R9; Mfr Part Nr (none) -> MFR50SFTE52-8R2; Vendor MFR50SFTE52-8R2 -> (none)
- R25: value 10R -> 4R99; Mfr Part Nr (none) -> CPF110R000BHE14; Vendor CPF110R000BHE14 -> (none)
- R26, R29: Mfr Part Nr (none) -> MFR50SFTE52-100R; Vendor MFR50SFTE52-100R -> (none)
- R27, R30, R8: Mfr Part Nr (none) -> MBB02070C4702FCT00; Vendor MBB02070C4702FCT00 -> (none)
- R28: Mfr Part Nr (none) -> MBB02070C4701FCT00; Vendor MBB02070C4701FCT00 -> (none)
- R3, R4: Mfr Part Nr (none) -> CPF110R000FEB14; Vendor CPF110R000FEB14 -> (none)
- R5, R6: Mfr Part Nr (none) -> CMF556K8100BEEK; Vendor CMF556K8100BEEK -> (none)
- SW1, SW2: Mfr Part Nr (none) -> PBH2UEESNPNAGX; Vendor PBH2UEEKZXNAG1RBLK -> (none)
- SW3: Mfr Part Nr (none) -> SR2612F-0112; Vendor Alpha -> (none)
- U1: value THAT1510P08-U -> 1512P08-U; Mfr Part Nr (none) -> 1512P08-U; Vendor THAT Corp -> (none)
Other:
- note added: "J3,J9 Mount either XLR or Jack"
- note added: "To calculate gain values, use micpre_gain2res.m with Octave. Example used here: [R_real, G_real, err] = micpre_gain2res([0 10 15:5:60], 'that1512', 'e96');"
- note removed: "Mount either one dual-color LED, or two single LEDs."
- note removed: "To calculate gain values, use micpre_gain2res.m with Octave. Example used here: [R_real, G_real, err] = micpre_gain2res([0 10 15:5:60], 'that1510', 'e12');"

Commit message: Rack: Correct gain resistor part numbers
Parts:
- R14: Mfr Part Nr MBB02070C1004FCT00 -> MFR50SFTE52-8K06
- R15: Mfr Part Nr MBB02070C2701FC100 -> MFR50SFTE52-909R
- R16: Mfr Part Nr MBB02070C1001FC100 -> MFR50SFTE52-453R
- R17: Mfr Part Nr MBB02070C5600FC100 -> MFR50SFTE52-237R
- R18: Mfr Part Nr MBB02070C2700FC100 -> MFR50SFTE52-127R
- R19: Mfr Part Nr MBB02070C1500FC100 -> MFR50SFTE52-71R
- R20: Mfr Part Nr MFR50SFTE52-82R -> MFR50SFTE52-39R
- R21: Mfr Part Nr MFR50SFTE52-47R -> MFR50SFTE52-22R
- R22: Mfr Part Nr MFR50SFTE52-27R -> MFR50SFTE52-12R4
- R23: Mfr Part Nr MFR50SFTE52-15R -> MFR50SFTE52-6R81
- R24: Mfr Part Nr MFR50SFTE52-8R2 -> MFR50SFTE52-3R9
- R25: Mfr Part Nr CPF110R000BHE14 -> MFR50SFTE52-4R99
Other:
- note added: "Note: D15, D16 and D17 can be any value between 15V and 18V, but they should all be the same value."
- note added: "Note: Value of the 220u-63V capacitors are not critical. Anything larger than 100uF-63 will do just fine."
Changed lines of the file:
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@@
+    (effects (font (size 1.27 1.27)) (justify left bottom))
+  )
+  (text "Note: Value of the 220u-63V capacitors are not critical. Anything larger than 100uF-63 will do just fine."
+    (at 80.01 19.05 0)
+    (effects (font (size 1.27 1.27)) (justify left bottom))
+  )
+  (text "Note: D15, D16 and D17 can be any value between 15V and 18V,\nbut they should all be the same value."
+    (at 97.79 95.25 0)
     (effects (font (size 1.27 1.27)) (justify left bottom))
   )
@@
       (effects (font (size 1.27 1.27)) hide)
     )
-    (property "Mfr Part Nr" "CPF110R000BHE14" (id 5) (at 266.7 106.68 0)
+    (property "Mfr Part Nr" "MFR50SFTE52-4R99" (id 5) (at 266.7 106.68 0)
       (effects (font (size 1.27 1.27)) hide)
     )
@@
       (effects (font (size 1.27 1.27)) hide)
     )
-    (property "Mfr Part Nr" "MBB02070C2701FC100" (id 5) (at 236.22 78.74 0)
+    (property "Mfr Part Nr" "MFR50SFTE52-909R" (id 5) (at 236.22 78.74 0)
       (effects (font (size 1.27 1.27)) hide)
     )
@@
       (effects (font (size 1.27 1.27)) hide)
     )
-    (property "Mfr Part Nr" "MBB02070C1001FC100" (id 5) (at 243.84 81.28 0)
+    (property "Mfr Part Nr" "MFR50SFTE52-453R" (id 5) (at 243.84 81.28 0)
       (effects (font (size 1.27 1.27)) hide)
     )
@@
       (effects (font (size 1.27 1.27)) hide)
     )
-    (property "Mfr Part Nr" "MBB02070C5600FC100" (id 5) (at 251.46 83.82 0)
+    (property "Mfr Part Nr" "MFR50SFTE52-237R" (id 5) (at 251.46 83.82 0)
       (effects (font (size 1.27 1.27)) hide)
     )
@@
       (effects (font (size 1.27 1.27)) hide)
     )
-    (property "Mfr Part Nr" "MBB02070C2700FC100" (id 5) (at 259.08 86.36 0)
+    (property "Mfr Part Nr" "MFR50SFTE52-127R" (id 5) (at 259.08 86.36 0)
       (effects (font (size 1.27 1.27)) hide)
     )
@@
       (effects (font (size 1.27 1.27)) hide)
     )
-    (property "Mfr Part Nr" "MBB02070C1500FC100" (id 5) (at 266.7 88.9 0)
+    (property "Mfr Part Nr" "MFR50SFTE52-71R" (id 5) (at 266.7 88.9 0)
       (effects (font (size 1.27 1.27)) hide)
     )
@@
       (effects (font (size 1.27 1.27)) hide)
     )
-    (property "Mfr Part Nr" "MFR50SFTE52-82R" (id 5) (at 228.6 93.98 0)
+    (property "Mfr Part Nr" "MFR50SFTE52-39R" (id 5) (at 228.6 93.98 0)
       (effects (font (size 1.27 1.27)) hide)
     )
@@
       (effects (font (size 1.27 1.27)) hide)
     )
-    (property "Mfr Part Nr" "MFR50SFTE52-47R" (id 5) (at 236.22 96.52 0)
+    (property "Mfr Part Nr" "MFR50SFTE52-22R" (id 5) (at 236.22 96.52 0)
       (effects (font (size 1.27 1.27)) hide)
     )
@@
       (effects (font (size 1.27 1.27)) hide)
     )
-    (property "Mfr Part Nr" "MFR50SFTE52-27R" (id 5) (at 243.84 99.06 0)
+    (property "Mfr Part Nr" "MFR50SFTE52-12R4" (id 5) (at 243.84 99.06 0)
       (effects (font (size 1.27 1.27)) hide)
     )
@@
       (effects (font (size 1.27 1.27)) hide)
     )
-    (property "Mfr Part Nr" "MFR50SFTE52-15R" (id 5) (at 251.46 101.6 0)
+    (property "Mfr Part Nr" "MFR50SFTE52-6R81" (id 5) (at 251.46 101.6 0)
       (effects (font (size 1.27 1.27)) hide)
     )
@@
       (effects (font (size 1.27 1.27)) hide)
     )
-    (property "Mfr Part Nr" "MFR50SFTE52-8R2" (id 5) (at 259.08 104.14 0)
+    (property "Mfr Part Nr" "MFR50SFTE52-3R9" (id 5) (at 259.08 104.14 0)
       (effects (font (size 1.27 1.27)) hide)
     )
@@
       (effects (font (size 1.27 1.27)) hide)
     )
-    (property "Mfr Part Nr" "MBB02070C1004FCT00" (id 5) (at 228.6 76.2 0)
-      (effects (font (size 1.27 1.27)) hide)
-    )
+    (property "Mfr Part Nr" "MFR50SFTE52-8K06" (id 5) (at 228.6 76.2 0)
+      (effects (font (size 1.27 1.27)) hide)
+    )
